File: eagle.sch (EAGLE design)
At the start: 26 parts, among them Q2 2N2222, T1 2N2222, U1 PIC16F877P

Commit message: Update eagle.sch
Parts:
- added X1: (no value), con-ptr500:AK300/2
- renumbered LED3 to LED2, LED4 to LED1, T1 to Q1
Connections:
- net GND: now also X1-2.KL
- net VCC: now also X1-1.KL
Changed lines of the file:
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@@
 <part name="D1" library="special" deviceset="7SEG-CK" device=""/>
 <part name="D2" library="special" deviceset="7SEG-CK" device=""/>
-<part name="T1" library="transistor" deviceset="2N2222" device=""/>
+<part name="Q1" library="transistor" deviceset="2N2222" device=""/>
 <part name="Q2" library="transistor" deviceset="2N2222" device=""/>
 <part name="AMPLIOP" library="ic-package" deviceset="DIL8" device=""/>
@@
 <part name="R1" library="rcl" deviceset="R-EU_" device="0204/7" value="10k"/>
 <part name="R5" library="rcl" deviceset="R-EU_" device="0204/7" value="280"/>
-<part name="LED4" library="eagle-ltspice" deviceset="LED_E" device="LD260"/>
-<part name="LED3" library="eagle-ltspice" deviceset="LED_E" device="LD260"/>
+<part name="LED1" library="eagle-ltspice" deviceset="LED_E" device="LD260"/>
+<part name="LED2" library="eagle-ltspice" deviceset="LED_E" device="LD260"/>
+<part name="X1" library="con-ptr500" library_urn="urn:adsk.eagle:library:181" deviceset="AK300/2" device="" package3d_urn="urn:adsk.eagle:package:9881/1"/>
 </parts>
 <sheets>
@@
 <instance part="D1" gate="G$1" x="157.48" y="30.48" smashed="yes"/>
 <instance part="D2" gate="G$1" x="180.34" y="15.24" smashed="yes"/>
-<instance part="T1" gate="G$1" x="154.94" y="-5.08" smashed="yes"/>
+<instance part="Q1" gate="G$1" x="154.94" y="-5.08" smashed="yes"/>
 <instance part="Q2" gate="G$1" x="175.26" y="-12.7" smashed="yes"/>
 <instance part="AMPLIOP" gate="G$1" x="25.4" y="129.54" smashed="yes"/>
@@
 <instance part="R1" gate="G$1" x="5.08" y="83.82" smashed="yes" rot="R90"/>
 <instance part="R5" gate="G$1" x="88.9" y="116.84" smashed="yes" rot="R90"/>
-<instance part="LED4" gate="G$1" x="76.2" y="134.62" smashed="yes" rot="R180"/>
-<instance part="LED3" gate="G$1" x="88.9" y="134.62" smashed="yes" rot="R180"/>
+<instance part="LED1" gate="G$1" x="76.2" y="134.62" smashed="yes" rot="R180"/>
+<instance part="LED2" gate="G$1" x="88.9" y="134.62" smashed="yes" rot="R180"/>
+<instance part="X1" gate="-1" x="0" y="45.72" smashed="yes">
+<attribute name="NAME" x="-1.27" y="46.609" size="1.778" layer="95" rot="R180"/>
+</instance>
+<instance part="X1" gate="-2" x="0" y="40.64" smashed="yes">
+<attribute name="NAME" x="-1.27" y="41.529" size="1.778" layer="95" rot="R180"/>
+<attribute name="VALUE" x="-3.81" y="36.957" size="1.778" layer="96"/>
+</instance>
 </instances>
 <busses>
@@
 <wire x1="76.2" y1="121.92" x2="76.2" y2="132.08" width="0.1524" layer="91"/>
 <pinref part="R4" gate="G$1" pin="2"/>
-<pinref part="LED4" gate="G$1" pin="A"/>
+<pinref part="LED1" gate="G$1" pin="A"/>
 </segment>
 </net>
@@
 <wire x1="165.1" y1="25.4" x2="165.1" y2="2.54" width="0.1524" layer="91"/>
 <wire x1="165.1" y1="2.54" x2="157.48" y2="2.54" width="0.1524" layer="91"/>
-<pinref part="T1" gate="G$1" pin="C"/>
+<pinref part="Q1" gate="G$1" pin="C"/>
 <wire x1="157.48" y1="2.54" x2="157.48" y2="0" width="0.1524" layer="91"/>
 </segment>
@@
 <pinref part="R5" gate="G$1" pin="2"/>
 <wire x1="88.9" y1="121.92" x2="88.9" y2="132.08" width="0.1524" layer="91"/>
-<pinref part="LED3" gate="G$1" pin="A"/>
+<pinref part="LED2" gate="G$1" pin="A"/>
 </segment>
 </net>
@@
 <wire x1="17.78" y1="119.38" x2="0" y2="119.38" width="0.1524" layer="91"/>
 <junction x="0" y="119.38"/>
-<label x="0" y="111.76" size="1.778" layer="95"/>
+<label x="-2.54" y="111.76" size="1.778" layer="95"/>
 </segment>
 <segment>
 <junction x="76.2" y="152.4"/>
-<pinref part="LED3" gate="G$1" pin="C"/>
+<pinref part="LED2" gate="G$1" pin="C"/>
 <wire x1="88.9" y1="139.7" x2="88.9" y2="152.4" width="0.1524" layer="91"/>
 <wire x1="88.9" y1="152.4" x2="76.2" y2="152.4" width="0.1524" layer="91"/>
-<pinref part="LED4" gate="G$1" pin="C"/>
+<pinref part="LED1" gate="G$1" pin="C"/>
 <wire x1="76.2" y1="139.7" x2="76.2" y2="152.4" width="0.1524" layer="91"/>
 <wire x1="76.2" y1="152.4" x2="50.8" y2="152.4" width="0.1524" layer="91"/>
@@
 <wire x1="5.08" y1="60.96" x2="5.08" y2="58.42" width="0.1524" layer="91"/>
 <junction x="5.08" y="60.96"/>
-<label x="5.08" y="53.34" size="1.778" layer="95"/>
+<label x="2.54" y="55.88" size="1.778" layer="95"/>
 </segment>
 <segment>
@@
 <wire x1="104.14" y1="17.78" x2="101.6" y2="17.78" width="0.1524" layer="91"/>
 <wire x1="101.6" y1="17.78" x2="101.6" y2="2.54" width="0.1524" layer="91"/>
-<label x="101.6" y="0" size="1.778" layer="95"/>
+<label x="99.06" y="0" size="1.778" layer="95"/>
 </segment>
 <segment>
@@
 <wire x1="177.8" y1="-17.78" x2="177.8" y2="-20.32" width="0.1524" layer="91"/>
 <wire x1="177.8" y1="-22.86" x2="177.8" y2="-20.32" width="0.1524" layer="91"/>
-<pinref part="T1" gate="G$1" pin="E"/>
+<pinref part="Q1" gate="G$1" pin="E"/>
 <wire x1="157.48" y1="-10.16" x2="162.56" y2="-10.16" width="0.1524" layer="91"/>
 <wire x1="162.56" y1="-10.16" x2="162.56" y2="-20.32" width="0.1524" layer="91"/>
 <wire x1="162.56" y1="-20.32" x2="177.8" y2="-20.32" width="0.1524" layer="91"/>
 <junction x="177.8" y="-20.32"/>
-<label x="177.8" y="-25.4" size="1.778" layer="95"/>
+<label x="175.26" y="-25.4" size="1.778" layer="95"/>
 </segment>
 <segment>
@@
 <wire x1="63.5" y1="35.56" x2="60.96" y2="35.56" width="0.1524" layer="91"/>
 <junction x="60.96" y="35.56"/>
-<label x="60.96" y="0" size="1.778" layer="95"/>
+<label x="58.42" y="0" size="1.778" layer="95"/>
+</segment>
+<segment>
+<pinref part="X1" gate="-2" pin="KL"/>
+<wire x1="5.08" y1="40.64" x2="10.16" y2="40.64" width="0.1524" layer="91"/>
+<label x="10.16" y="40.64" size="1.778" layer="91"/>
 </segment>
 </net>
@@
 <pinref part="U1" gate="G$1" pin="RE0/!RD/AN5"/>
 <wire x1="40.64" y1="73.66" x2="30.48" y2="73.66" width="0.1524" layer="91"/>
-<pinref part="T1" gate="G$1" pin="B"/>
+<pinref part="Q1" gate="G$1" pin="B"/>
 <wire x1="30.48" y1="73.66" x2="30.48" y2="-5.08" width="0.1524" layer="91"/>
 <wire x1="30.48" y1="-5.08" x2="152.4" y2="-5.08" width="0.1524" layer="91"/>
@@
 <wire x1="-5.08" y1="137.16" x2="5.08" y2="137.16" width="0.1524" layer="91"/>
 <wire x1="5.08" y1="137.16" x2="5.08" y2="144.78" width="0.1524" layer="91"/>
-<label x="5.08" y="147.32" size="1.778" layer="95"/>
+<label x="2.54" y="144.78" size="1.778" layer="95"/>
 </segment>
 <segment>
 <pinref part="R1" gate="G$1" pin="2"/>
 <wire x1="5.08" y1="88.9" x2="5.08" y2="91.44" width="0.1524" layer="91"/>
-<label x="0" y="91.44" size="1.778" layer="95"/>
+<label x="2.54" y="91.44" size="1.778" layer="95"/>
 </segment>
 <segment>
@@
 <wire x1="101.6" y1="20.32" x2="101.6" y2="22.86" width="0.1524" layer="91"/>
 <junction x="101.6" y="22.86"/>
-<label x="93.98" y="22.86" size="1.778" layer="95"/>
+<label x="93.98" y="20.32" size="1.778" layer="95"/>
 </segment>
 <segment>
 <pinref part="C7" gate="G$1" pin="2"/>
 <wire x1="104.14" y1="101.6" x2="104.14" y2="106.68" width="0.1524" layer="91"/>
-<label x="104.14" y="106.68" size="1.778" layer="95"/>
+<label x="101.6" y="106.68" size="1.778" layer="95"/>
 </segment>
 <segment>
@@
 <wire x1="60.96" y1="114.3" x2="60.96" y2="127" width="0.1524" layer="91"/>
 <wire x1="60.96" y1="114.3" x2="60.96" y2="101.6" width="0.1524" layer="91"/>
-<label x="60.96" y="132.08" size="1.778" layer="95"/>
+<label x="58.42" y="127" size="1.778" layer="95"/>
 </segment>
 <segment>
@@
 <wire x1="33.02" y1="129.54" x2="40.64" y2="129.54" width="0.1524" layer="91"/>
 <label x="40.64" y="129.54" size="1.778" layer="95"/>
+</segment>
+<segment>
+<pinref part="X1" gate="-1" pin="KL"/>
+<wire x1="5.08" y1="45.72" x2="10.16" y2="45.72" width="0.1524" layer="91"/>
+<label x="10.16" y="45.72" size="1.778" layer="91"/>
 </segment>
 </net>
@@
 </schematic>
 </drawing>
+<compatibility>
+<note version="8.2" severity="warning">
+Since Version 8.2, EAGLE supports online libraries. The ids
+of those online libraries will not be understood (or retained)
+with this version.
+</note>
+<note version="8.3" severity="warning">
+Since Version 8.3, EAGLE supports URNs for individual library
+assets (packages, symbols, and devices). The URNs of those assets
+will not be understood (or retained) with this version.
+</note>
+<note version="8.3" severity="warning">
+Since Version 8.3, EAGLE supports the association of 3D packages
+with devices in libraries, schematics, and board files. Those 3D
+packages will not be understood (or retained) with this version.
+</note>
+</compatibility>
 </eagle>
