File: ElecBoardv3.brd (EAGLE design)
At the start: 100 x 80 mm, 27 parts, among them Q1 2N2222, Q2 2N2222, U1 PIC16F877P

Commit message: Last update 97,3% (opt 4)
Other:
- board text removed: "Groupe 3 Almasy Zita, Bohyn Gauthier, Hermant Thibaut, Ponjée Aymeric"
Changed lines of the file:
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@@
 <wire x1="100" y1="80" x2="0" y2="80" width="0" layer="20"/>
 <wire x1="0" y1="80" x2="0" y2="0" width="0" layer="20"/>
-<text x="2.54" y="81.28" size="1.778" layer="1">Groupe 3
-Almasy Zita, Bohyn Gauthier, Hermant Thibaut, Ponjée Aymeric </text>
 </plain>
 <attributes>
@@
 <param name="PrefDir.14" value="0"/>
 <param name="PrefDir.15" value="0"/>
-<param name="PrefDir.16" value="-"/>
+<param name="PrefDir.16" value="a"/>
 <param name="cfVia" value="8"/>
 <param name="cfNonPref" value="5"/>
@@
 <contactref element="C2" pad="2"/>
 <wire x1="11.43" y1="43.18" x2="20.32" y2="46.99" width="0" layer="19" extent="1-1"/>
-<wire x1="31.75" y1="20.32" x2="11.43" y2="43.18" width="0" layer="19" extent="1-1"/>
+<wire x1="31.75" y1="20.32" x2="20.32" y2="46.99" width="0" layer="19" extent="1-1"/>
 </signal>
 <signal name="N$8">
@@
 <contactref element="R4" pad="1"/>
 <contactref element="U1" pad="15"/>
-<wire x1="31.75" y1="17.78" x2="12.7" y2="19.05" width="0" layer="19" extent="1-1"/>
+<wire x1="12.7" y1="19.05" x2="31.75" y2="17.78" width="0" layer="19" extent="1-1"/>
 </signal>
 <signal name="N$9">
@@
 <contactref element="Q1" pad="3"/>
 <wire x1="72.39" y1="15.24" x2="72.39" y2="30.48" width="0" layer="19" extent="1-1"/>
-<wire x1="54.61" y1="46.99" x2="72.39" y2="15.24" width="0" layer="19" extent="1-1"/>
+<wire x1="54.61" y1="46.99" x2="72.39" y2="30.48" width="0" layer="19" extent="1-1"/>
 </signal>
 <signal name="N$47">
@@
 <contactref element="R5" pad="2"/>
 <contactref element="LED2" pad="A"/>
-<wire x1="21.59" y1="25.4" x2="22.86" y2="21.59" width="0" layer="19" extent="1-1"/>
+<wire x1="22.86" y1="21.59" x2="21.59" y2="25.4" width="0" layer="19" extent="1-1"/>
 </signal>
 <signal name="COMPIM">
@@
 <contactref element="U1" pad="12"/>
 <contactref element="X1" pad="2"/>
-<wire x1="46.99" y1="30.48" x2="66.04" y2="50.8" width="0" layer="19" extent="1-1"/>
+<wire x1="57.15" y1="49.53" x2="66.04" y2="50.8" width="0" layer="19" extent="1-1"/>
+<wire x1="46.99" y1="30.48" x2="57.15" y2="49.53" width="0" layer="19" extent="1-1"/>
 <wire x1="54.61" y1="17.78" x2="46.99" y2="30.48" width="0" layer="19" extent="1-1"/>
 <wire x1="31.75" y1="25.4" x2="46.99" y2="30.48" width="0" layer="19" extent="1-1"/>
-<wire x1="57.15" y1="49.53" x2="54.61" y2="17.78" width="0" layer="19" extent="1-1"/>
-<wire x1="92.71" y1="13.97" x2="57.15" y2="49.53" width="0" layer="19" extent="1-1"/>
 <wire x1="21.59" y1="27.94" x2="31.75" y2="25.4" width="0" layer="19" extent="1-1"/>
 <wire x1="12.7" y1="34.29" x2="21.59" y2="27.94" width="0" layer="19" extent="1-1"/>
+<wire x1="19.05" y1="39.37" x2="12.7" y2="34.29" width="0" layer="19" extent="1-1"/>
 <wire x1="8.89" y1="43.18" x2="12.7" y2="34.29" width="0" layer="19" extent="1-1"/>
-<wire x1="19.05" y1="39.37" x2="12.7" y2="34.29" width="0" layer="19" extent="1-1"/>
-<wire x1="12.7" y1="55.88" x2="19.05" y2="39.37" width="0" layer="19" extent="1-1"/>
+<wire x1="12.7" y1="55.88" x2="8.89" y2="43.18" width="0" layer="19" extent="1-1"/>
 <wire x1="11.7094" y1="64.0588" x2="12.7" y2="55.88" width="0" layer="19" extent="1-1"/>
 <wire x1="11.7094" y1="70.5612" x2="11.7094" y2="64.0588" width="0" layer="19" extent="1-1"/>
-<wire x1="22.86" y1="54.61" x2="11.7094" y2="64.0588" width="0" layer="19" extent="1-1"/>
+<wire x1="22.86" y1="54.61" x2="12.7" y2="55.88" width="0" layer="19" extent="1-1"/>
 <wire x1="34.29" y1="60.96" x2="22.86" y2="54.61" width="0" layer="19" extent="1-1"/>
 <wire x1="36.83" y1="76.2" x2="34.29" y2="60.96" width="0" layer="19" extent="1-1"/>
 <wire x1="12.7" y1="10.1092" x2="21.59" y2="27.94" width="0" layer="19" extent="1-1"/>
+<wire x1="92.71" y1="13.97" x2="54.61" y2="17.78" width="0" layer="19" extent="1-1"/>
 </signal>
 <signal name="N$26">
@@
 <contactref element="MAX232" pad="2"/>
 <contactref element="C7" pad="1"/>
-<wire x1="72.39" y1="68.58" x2="54.61" y2="66.04" width="0" layer="19" extent="1-1"/>
+<wire x1="54.61" y1="66.04" x2="72.39" y2="68.58" width="0" layer="19" extent="1-1"/>
 </signal>
 <signal name="N$18">
@@
 <contactref element="U1" pad="1"/>
 <wire x1="31.75" y1="53.34" x2="38.1" y2="64.77" width="0" layer="19" extent="1-1"/>
-<wire x1="16.2306" y1="64.0588" x2="38.1" y2="64.77" width="0" layer="19" extent="1-1"/>
+<wire x1="15.24" y1="55.88" x2="31.75" y2="53.34" width="0" layer="19" extent="1-1"/>
+<wire x1="16.2306" y1="64.0588" x2="15.24" y2="55.88" width="0" layer="19" extent="1-1"/>
 <wire x1="16.2306" y1="70.5612" x2="16.2306" y2="64.0588" width="0" layer="19" extent="1-1"/>
-<wire x1="15.24" y1="55.88" x2="16.2306" y2="64.0588" width="0" layer="19" extent="1-1"/>
 </signal>
 <signal name="N$30">
@@
 <contactref element="U1" pad="2"/>
 <wire x1="27.94" y1="67.31" x2="39.37" y2="68.58" width="0" layer="19" extent="1-1"/>
-<wire x1="31.75" y1="50.8" x2="39.37" y2="68.58" width="0" layer="19" extent="1-1"/>
+<wire x1="31.75" y1="50.8" x2="27.94" y2="67.31" width="0" layer="19" extent="1-1"/>
 </signal>
 <signal name="N$33">
@@
 <wire x1="54.61" y1="20.32" x2="54.61" y2="22.86" width="0" layer="19" extent="1-1"/>
 <wire x1="31.75" y1="27.94" x2="46.99" y2="33.02" width="0" layer="19" extent="1-1"/>
+<wire x1="24.13" y1="39.37" x2="31.75" y2="27.94" width="0" layer="19" extent="1-1"/>
 <wire x1="12.7" y1="5.1054" x2="31.75" y2="27.94" width="0" layer="19" extent="1-1"/>
-<wire x1="24.13" y1="39.37" x2="31.75" y2="27.94" width="0" layer="19" extent="1-1"/>
 </signal>
 </signals>
@@
 </drawing>
 <compatibility>
-<note version="6.3" minversion="6.2.2" severity="warning">
-Since Version 6.2.2 text objects can contain more than one line,
-which will not be processed correctly with this version.
-</note>
 <note version="8.2" severity="warning">
 Since Version 8.2, EAGLE supports online libraries. The ids
