File: Final/Groupe3_Hermant-Bohyn-Almasy-Ponjee.brd (EAGLE design)
At the start: 100 x 80 mm, 27 parts, among them Q1 2N2222, Q2 2N2222, U1 PIC16F877P

Commit message: Add files via upload
Routing:
- net N$35: track 33.4 -> 51.9 mm
- net GND: track 331.5 -> 333.3 mm
Changed lines of the file:
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@@
 <layer number="27" name="tValues" color="7" fill="1" visible="yes" active="yes"/>
 <layer number="28" name="bValues" color="7" fill="1" visible="yes" active="yes"/>
-<layer number="29" name="tStop" color="7" fill="3" visible="no" active="yes"/>
-<layer number="30" name="bStop" color="7" fill="6" visible="no" active="yes"/>
+<layer number="29" name="tStop" color="7" fill="3" visible="yes" active="yes"/>
+<layer number="30" name="bStop" color="7" fill="6" visible="yes" active="yes"/>
 <layer number="31" name="tCream" color="7" fill="4" visible="no" active="yes"/>
 <layer number="32" name="bCream" color="7" fill="5" visible="no" active="yes"/>
@@
 <wire x1="0" y1="80" x2="0" y2="0" width="0" layer="20"/>
 <text x="12.7" y="76.2" size="1.778" layer="16" rot="MR0">Groupe 3</text>
+<rectangle x1="30.48" y1="68.326" x2="34.29" y2="71.628" layer="16"/>
 </plain>
 <attributes>
@@
 <wire x1="8.89" y1="43.18" x2="12.7" y2="39.37" width="0.381" layer="16"/>
 <wire x1="7.62" y1="33.655" x2="7.62" y2="16.51" width="0.381" layer="16"/>
-<wire x1="5.334" y1="16.51" x2="5.334" y2="7.4168" width="0.381" layer="16"/>
-<wire x1="5.334" y1="7.4168" x2="7.62" y2="5.1308" width="0.381" layer="16"/>
+<wire x1="4.064" y1="16.51" x2="4.064" y2="8.6868" width="0.381" layer="16"/>
+<wire x1="4.064" y1="8.6868" x2="7.62" y2="5.1308" width="0.381" layer="16"/>
 <wire x1="12.7" y1="38.735" x2="7.62" y2="33.655" width="0.381" layer="16"/>
 <wire x1="33.655" y1="20.955" x2="33.02" y2="21.59" width="0.381" layer="16"/>
 <wire x1="33.655" y1="17.145" x2="33.655" y2="20.955" width="0.381" layer="16"/>
 <wire x1="33.02" y1="16.51" x2="33.655" y2="17.145" width="0.381" layer="16"/>
-<wire x1="5.334" y1="16.51" x2="7.62" y2="16.51" width="0.381" layer="16"/>
+<wire x1="4.064" y1="16.51" x2="7.62" y2="16.51" width="0.381" layer="16"/>
 <wire x1="7.62" y1="16.51" x2="33.02" y2="16.51" width="0.381" layer="16"/>
 <wire x1="12.7" y1="46.99" x2="12.7" y2="55.88" width="0.381" layer="16"/>
@@
 <contactref element="AMPLIOP" pad="6"/>
 <contactref element="U1" pad="2"/>
-<wire x1="35.56" y1="67.31" x2="27.94" y2="67.31" width="0.381" layer="16"/>
+<wire x1="35.56" y1="67.31" x2="31.75" y2="67.31" width="0.381" layer="16"/>
+<wire x1="31.75" y1="67.31" x2="27.94" y2="67.31" width="0.381" layer="16"/>
 <wire x1="36.195" y1="66.675" x2="35.56" y2="67.31" width="0.381" layer="16"/>
-<wire x1="37.465" y1="66.675" x2="36.195" y2="66.675" width="0.381" layer="16"/>
-<wire x1="39.37" y1="68.58" x2="37.465" y2="66.675" width="0.381" layer="16"/>
 <wire x1="39.37" y1="58.42" x2="31.75" y2="50.8" width="0.381" layer="16"/>
 <wire x1="39.37" y1="68.58" x2="39.37" y2="58.42" width="0.381" layer="16"/>
+<wire x1="39.37" y1="68.58" x2="37.465" y2="66.675" width="0.381" layer="16"/>
+<wire x1="37.465" y1="66.675" x2="36.195" y2="66.675" width="0.381" layer="16"/>
+<wire x1="39.37" y1="68.58" x2="35.56" y2="64.77" width="0.381" layer="16"/>
+<wire x1="35.56" y1="64.77" x2="31.496" y2="64.77" width="0.381" layer="16"/>
+<wire x1="39.37" y1="68.58" x2="34.29" y2="63.5" width="0.381" layer="16"/>
+<wire x1="34.29" y1="63.5" x2="33.9697" y2="63.5" width="0.381" layer="16"/>
+<wire x1="31.75" y1="67.31" x2="31.75" y2="68.834" width="0.381" layer="16"/>
 </signal>
 <signal name="N$33">
@@
 <wire x1="52.07" y1="66.04" x2="62.23" y2="76.2" width="0.381" layer="16"/>
 </signal>
+<signal name="S$1">
+<via x="31.242" y="64.77" extent="1-16" drill="0.35"/>
+</signal>
+<signal name="S$2">
+<via x="34.036" y="63.5" extent="1-16" drill="0.35"/>
+</signal>
 </signals>
