File: Final/Final/Groupe3_Hermant-Bohyn-Almasy-Ponjee.brd (EAGLE design)
At the start: 100 x 80 mm, 27 parts, among them Q1 2N2222, Q2 2N2222, U1 PIC16F877P

Commit message: Add files via upload
Parts:
- C7: value 100u -> 10uF
Changed lines of the file:
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@@
 <attribute name="VALUE" x="62.23" y="54.356" size="1.27" layer="27" ratio="10" rot="R270"/>
 </element>
-<element name="C7" library="rcl" package="C025-050X050" value="100u" x="53.34" y="66.04" smashed="yes" rot="R180">
+<element name="C7" library="rcl" package="C025-050X050" value="10uF" x="53.34" y="66.04" smashed="yes" rot="R180">
 <attribute name="NAME" x="55.626" y="63.5" size="1.27" layer="25" ratio="10" rot="R180"/>
 <attribute name="VALUE" x="55.626" y="69.85" size="1.27" layer="27" ratio="10" rot="R180"/>
