File: Final/Final/Groupe3_Hermant-Bohyn-Almasy-Ponjee.sch (EAGLE design)
At the start: 27 parts, among them Q1 2N2222, Q2 2N2222, U1 PIC16F877P

Commit message: Add files via upload
Parts:
- C7: value 100u -> 10uF
Changed lines of the file:
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@@
 <part name="MAX232" library="ic-package" deviceset="DIL16" device=""/>
 <part name="C61" library="rcl" deviceset="C-EU" device="025-050X050" value="10uF"/>
-<part name="C7" library="rcl" deviceset="C-EU" device="025-050X050" value="100u"/>
+<part name="C7" library="rcl" deviceset="C-EU" device="025-050X050" value="10uF"/>
 <part name="P1/COMPIM" library="con-subd" deviceset="F09" device="V"/>
 <part name="4511" library="ic-package" deviceset="DIL16" device=""/>
